File: hardware/prj-kicad/cowstick-ums.kicad_pcb (KiCad board)
At the start: 2 copper layers, 45 x 19 mm, 12 parts, among them J1 CONN_USB-A, U2 LM3671, U90 AZ2210

Commit message: Hardware: Improve PCB r1, add MCU (STM32G0)
Parts:
- added C5: 100nF, cowstick-ums:C_0603, F.Cu at (142.2, 105.0)
- added C6: 1uF, cowstick-ums:C_0603, F.Cu at (141.5, 108.0)
- added C7: 12.5pF, cowstick-ums:C_0603, F.Cu at (139.2, 100.0)
- added C8: 12.5pF, cowstick-ums:C_0603, F.Cu at (143.2, 100.0)
- added R1: 10k, cowstick-ums:R_0603, F.Cu at (140.0, 108.0)
- added U1: STM32G0KxT, cowstick-ums:TQFP32, F.Cu at (148.5, 105.0)
- added X1: 32,768k, cowstick-ums:Q_3.2x1.5, F.Cu at (141.2, 102.0)
- moved C3 0.25 mm to (140.0, 111.8)
- moved C4 0.25 mm to (142.0, 111.8)
Routing:
- net GND: track 73.7 -> 99.2 mm, vias 28 -> 35
- net +3.3V: track 15.2 -> 40.0 mm, vias 1 -> 6
- net USB_DP: track 0.00 -> 14.8 mm, vias 0 -> 2
- net USB_DM: track 0.00 -> 14.6 mm, vias 0 -> 2
- net Net-(U1-Pad3): track 0.00 -> 7.25 mm
- net RST: track 0.00 -> 4.68 mm
- net Net-(C8-Pad1): track 0.00 -> 4.32 mm
- net +VBus: track 22.7 -> 22.8 mm, vias 2 -> 7
- added copper zone on In2.Cu, net +3.3V
- added copper zone on In2.Cu, net +VBus
- added copper zone on In1.Cu, net GND
Other:
- copper layers 2 -> 4
- board text removed: "MCU"

Commit message: Hardware: Improve PCB r1, add two SOIC8 flash memory ic for channel 1
Parts:
- added C10: 100nF, cowstick-ums:C_0603, F.Cu at (163.3, 104.8)
- added C9: 100nF, cowstick-ums:C_0603, F.Cu at (158.3, 104.0)
- added U3: W25QxxVSN, cowstick-ums:SOIC-8, F.Cu at (159.5, 109.2)
- added U4: W25QxxVSN, cowstick-ums:SOIC-8, F.Cu at (167.0, 109.2)
Connections:
- U1 pad 16: unconnected-(U1-Pad16) -> SPI1_CS2
- U1 pad 17: unconnected-(U1-Pad17) -> SPI1_WP
- U1 pad 18: unconnected-(U1-Pad18) -> SPI1_HLD
Routing:
- net GND: track 99.2 -> 146.6 mm, vias 35 -> 52
- net +3.3V: track 40.0 -> 71.7 mm, vias 6 -> 8
- net SPI1_MISO: track 0.00 -> 25.0 mm, vias 0 -> 3
- net SPI1_SCK: track 0.00 -> 25.0 mm, vias 0 -> 3
- net SPI1_MOSI: track 0.00 -> 24.3 mm, vias 0 -> 3
- net SPI1_CS2: track 0.00 -> 22.8 mm, vias 0 -> 2
- net SPI1_WP: track 0.00 -> 20.9 mm
- net SPI1_HLD: track 0.00 -> 19.4 mm
- net SPI1_CS1: track 0.00 -> 15.3 mm, vias 0 -> 2
Other:
- board text removed: "Mem1"

Commit message: Hardware: Improve PCB r1, add one Nand flash memory for "large" capacity (channel 2)
Parts:
- added C11: 100nF, cowstick-ums:C_0603, F.Cu at (167.6, 98.2)
- added U5: W25NxxVZE, cowstick-ums:WSON8, F.Cu at (162.0, 99.5)
Connections:
- U1 pad 1: unconnected-(U1-Pad1) -> SPI2_CS
Routing:
- net GND: track 146.6 -> 212.1 mm, vias 52 -> 80
- net SPI2_SCK: track 0.00 -> 25.0 mm, vias 0 -> 2
- net SPI2_MOSI: track 0.00 -> 25.0 mm, vias 0 -> 2
- net SPI2_CS: track 0.00 -> 24.8 mm, vias 0 -> 2
- net SPI2_MISO: track 0.00 -> 24.7 mm, vias 0 -> 2
- net +3.3V: track 71.7 -> 89.7 mm, vias 8 -> 9
Other:
- board text removed: "Mem2"

Commit message: Hardware: Finish and cleanup pcb r1 and create production files
Parts:
- added D2: LED, cowstick-ums:C_0805, F.Cu at (146.0, 97.5)
- added R4: 330, cowstick-ums:R_0603, F.Cu at (142.5, 97.2)
- added TP1: CONN_1, cowstick-ums:TP_SMD, F.Cu at (144.0, 111.0)
- added TP2: CONN_1, cowstick-ums:TP_SMD, B.Cu at (154.1, 105.8)
- added TP3: CONN_1, cowstick-ums:TP_SMD, B.Cu at (146.5, 105.8)
- added TP4: CONN_1, cowstick-ums:TP_SMD, B.Cu at (149.0, 105.8)
- added TP5: CONN_1, cowstick-ums:TP_SMD, B.Cu at (151.5, 105.8)
- added TP6: CONN_1, cowstick-ums:TP_PIN, F.Cu at (146.5, 112.5)
- added TP7: CONN_1, cowstick-ums:TP_PIN, F.Cu at (149.0, 112.5)
- added TP8: CONN_1, cowstick-ums:TP_PIN, F.Cu at (151.5, 112.5)
- added TP9: CONN_1, cowstick-ums:TP_PIN, F.Cu at (168.5, 103.0)
- added agilack-11.5: 450px, cowstick-ums:logo-agilack-11.5, F.Cu at (154.8, 105.0)
- added ohw_logo: VAL**, cowstick-ums:logo-ohw, F.Cu at (134.2, 100.7)
Connections:
- U1 pad 10: unconnected-(U1-Pad10) -> UART_RX
- U1 pad 24: Net-(TP5-Pad1) -> SWD_IO
- U1 pad 25: Net-(TP4-Pad1) -> SWD_CLK
- U1 pad 27: unconnected-(U1-Pad27) -> SPI2_HLD
- U1 pad 28: unconnected-(U1-Pad28) -> SPI2_WP
- U1 pad 29: unconnected-(U1-Pad29) -> LED
- U1 pad 9: unconnected-(U1-Pad9) -> UART_TX
- U5 pad 3: unconnected-(U5-Pad3) -> SPI2_WP
- U5 pad 7: unconnected-(U5-Pad7) -> SPI2_HLD
Routing:
- net GND: track 212.1 -> 243.4 mm, vias 80 -> 81
- net SPI2_HLD: track 0.00 -> 21.9 mm
- net SPI2_WP: track 0.00 -> 10.7 mm
- net +3.3V: track 89.7 -> 98.1 mm, vias 9 -> 11
- net UART_RX: track 0.00 -> 7.11 mm
- net SWD_CLK: track 0.00 -> 5.95 mm, vias 0 -> 1
- net SWD_IO: track 0.00 -> 5.52 mm, vias 0 -> 1
- net UART_TX: track 0.00 -> 5.24 mm
- net LED: track 0.00 -> 5.15 mm
- net RST: track 4.68 -> 7.08 mm, vias 0 -> 1
- net Net-(D2-Pad1): track 0.00 -> 1.89 mm
- added copper zone on B.Cu, net GND
Other:
- board text added: "(c) Agilack 2023"
- board text added: "Cowstick-UMS"
- board text added: "rev1"

Commit message: Hardware: Modify PCB for a new revision (rev2) and create production files  - Add pushbutton and a second LED  - Replace power reg and USB connector with a new refs
Parts:
- removed C90: 100pF, cowstick-ums:C_0603
- removed U90: AZ2210, cowstick-ums:SOT23-5
- added C12: 1uF, cowstick-ums:C_0603, F.Cu at (139.2, 98.2)
- added D3: LED, cowstick-ums:C_0805, F.Cu at (129.5, 97.8)
- added R5: R, cowstick-ums:R_0603, F.Cu at (136.8, 112.0)
- added R6: R, cowstick-ums:R_0603, F.Cu at (136.8, 113.5)
- added R7: 330, cowstick-ums:R_0603, F.Cu at (135.5, 97.5)
- added SW1: SW_PUSH, cowstick-ums:BUT_TC029, F.Cu at (134.8, 100.8)
- added TP10: CONN_1, cowstick-ums:TP_SMD, B.Cu at (130.2, 110.0)
- added TP11: CONN_1, cowstick-ums:TP_SMD, B.Cu at (130.2, 105.0)
- J1: footprint cowstick-ums:CONN_MC32604 -> cowstick-ums:CONN_AM90YC
- L1: footprint cowstick-ums:I_CDRH2D14 -> cowstick-ums:I_SMD_3x3
- TP1: footprint cowstick-ums:TP_SMD -> cowstick-ums:TP_SMD2
- TP7, TP8: footprint cowstick-ums:TP_PIN -> cowstick-ums:TP_SMD; moved to B.Cu
- U2: value LM3671 -> MT3410
- moved ohw_logo 22.2 mm to (153.8, 111.2)
- moved TP7 10.3 mm to (138.8, 110.8), turned to 180 degrees
- moved TP8 10.3 mm to (141.4, 110.8), turned to 180 degrees
- moved agilack-11.5 2.76 mm to (155.0, 102.2)
- moved D2 2.50 mm to (148.5, 97.5)
- moved L1 2.40 mm to (136.8, 109.5)
- moved R1 2.25 mm to (142.2, 108.0)
- moved C6 1.25 mm to (140.2, 108.0), turned to 90 degrees
- moved R4 1.25 mm to (143.2, 98.2)
- moved J1 0.65 mm to (127.6, 105.0)
- moved TP1 0.56 mm to (144.5, 111.2)
- moved U2 0.56 mm to (132.5, 111.5), turned to 90 degrees
- turned C3 to -90 degrees
- turned C4 to -90 degrees
Connections:
- L1 pad 1: Net-(L1-Pad1) -> /VSW
- U1 pad 7: unconnected-(U1-Pad7) -> BUTTON
- U1 pad 8: unconnected-(U1-Pad8) -> LED2
- U2 pad 3: +VBus -> /VSW
- U2 pad 4: +3.3V -> +VBus
- U2 pad 5: Net-(L1-Pad1) -> Net-(R5-Pad1)
Routing:
- net LED2: track 0.00 -> 23.7 mm, vias 0 -> 2
- net BUTTON: track 0.00 -> 18.2 mm, vias 0 -> 2
- net GND: track 243.4 -> 259.7 mm, vias 81 -> 78
- net +3.3V: track 98.1 -> 82.3 mm, vias 11 -> 8
- net Net-(R5-Pad1): track 0.00 -> 6.84 mm
- net Net-(D3-Pad1): track 0.00 -> 4.39 mm
- net +VBus: track 22.8 -> 25.1 mm
- net UART_TX: track 5.24 -> 7.51 mm, vias 0 -> 1
- net /VSW: track 0.00 -> 2.16 mm
- net Net-(L1-Pad1): track 2.01 -> 0.00 mm
- net Net-(D2-Pad1): track 1.89 -> 3.85 mm
- net LED: track 5.15 -> 3.81 mm
- net Net-(C90-Pad1): track 1.24 -> 0.00 mm
- net RST: track 7.08 -> 7.80 mm
- net UART_RX: track 7.11 -> 7.40 mm, vias 0 -> 1
- added copper zone on F.Cu, net /VSW
- removed copper zone on B.Cu, net +VBus
Other:
- board text added: "3V3"
- board text added: "GND"
- board text added: "RST"
- board text added: "RX"
- board text added: "SWCLK"
- board text added: "SWDIO"
- board text added: "TX"
- board text added: "VBUS"
- board text added: "rev2"
- board text removed: "rev1"
